Commit message: urdf改成麥克那母輪 機器學習能動了

File: esp32_receiver/description/gazebo_control.xacro (robot description, xacro)
@@ -3,5 +3,7 @@
     <xacro:macro name="gazebo_control" params="ns">
         <gazebo>
-            <plugin name="diff_drive" filename="libgazebo_ros_diff_drive.so">
+            <!-- <plugin name="diff_drive" filename="libgazebo_ros_diff_drive.so"> -->
+            <!-- <plugin name="mecanum_drive" filename="libgazebo_ros_mecanum_drive.so"> -->
+            <plugin name="mecanum_drive" filename="libgazebo_mecanum_drive.so">
                 <ros>
                     <namespace>${ns}</namespace>
@@ -16,22 +18,36 @@
                 <left_joint>back_left_wheel_joint</left_joint>
                 <right_joint>back_right_wheel_joint</right_joint> -->
-                <left_joint>left_wheel_joint</left_joint>
-                <right_joint>right_wheel_joint</right_joint>
-                <!-- <left_joint>back_right_wheel_joint</left_joint>
-                <right_joint>back_left_wheel_joint</right_joint> -->
+                <commandTopic>cmd_vel</commandTopic>
+                <odometryTopic>odom</odometryTopic>
+                <odometryFrame>odom</odometryFrame>
+                <robotBaseFrame>base_footprint</robotBaseFrame>
+                <LeftRear>back_left_wheel_joint</LeftRear>
+                <LeftFront>front_left_wheel_joint</LeftFront>
+                <RightFront>front_right_wheel_joint</RightFront>
+                <RightRear>back_right_wheel_joint</RightRear>
+                <odometryRate>20</odometryRate>
+                <publishWheelTF>true</publishWheelTF>
+                <publishWheelJointState>true</publishWheelJointState>
+                <WheelTorque>1</WheelTorque>
+                <WheelSeparationW>0.12</WheelSeparationW>
+                <WheelSeparationL>0.16</WheelSeparationL>
+                <wheelAccel>5</wheelAccel>
+                <wheelDiameter>0.03</wheelDiameter>
+                <publishOdom>true</publishOdom>
+                <isRollerModel>false</isRollerModel>
+                <!-- kinematics -->
                 <!-- <wheel_separation>0.35</wheel_separation>
+                <wheel_separation_x>0.35</wheel_separation_x>
+                <wheel_separation_y>0.25</wheel_separation_y>
                 <wheel_diameter>0.1</wheel_diameter> -->
-                <!-- kinematics -->
-                <wheel_separation>0.35</wheel_separation>
-                <wheel_diameter>0.1</wheel_diameter>
                 <!-- Limits -->
-                <max_wheel_torque>200</max_wheel_torque>
-                <max_wheel_acceleration>10.0</max_wheel_acceleration>
+                <!-- <max_wheel_torque>200</max_wheel_torque>
+                <max_wheel_acceleration>10.0</max_wheel_acceleration> -->
                 <!-- Output -->
-                <odometry_frame>odom</odometry_frame>
+                <!-- <odometry_frame>odom</odometry_frame>
                 <robot_base_frame>base_link</robot_base_frame>
                 <publish_odom>true</publish_odom>
                 <publish_odom_tf>true</publish_odom_tf>
-                <publish_wheel_tf>true</publish_wheel_tf>
+                <publish_wheel_tf>true</publish_wheel_tf> -->
             </plugin>
         </gazebo>

File: esp32_receiver/description/gazebo_table.urdf.xacro (robot description, xacro)
@@ -45,6 +45,31 @@
     <xacro:create_zone parent="wall5_link" offset_x="4" offset_y="-4" parent_two="wall5_link"/>
     <xacro:create_zone parent="wall6_link" offset_x="8" offset_y="-4" parent_two="wall6_link"/>
-    <!-- <xacro:create_zone parent="wall7_link" offset_x="0" offset_y="-8" parent_two="wall7_link"/>
+    <xacro:create_zone parent="wall7_link" offset_x="0" offset_y="-8" parent_two="wall7_link"/>
     <xacro:create_zone parent="wall8_link" offset_x="4" offset_y="-8" parent_two="wall8_link"/>
-    <xacro:create_zone parent="wall9_link" offset_x="8" offset_y="-8" parent_two="wall9_link"/> -->
+    <xacro:create_zone parent="wall9_link" offset_x="8" offset_y="-8" parent_two="wall9_link"/>
+    <!-- <xacro:create_zone parent="wall1_link" offset_x="0" offset_y="0" parent_two="wall1_link"/>
+    <xacro:create_zone parent="wall2_link" offset_x="4" offset_y="0" parent_two="wall2_link"/>
+    <xacro:create_zone parent="wall3_link" offset_x="8" offset_y="0" parent_two="wall3_link"/>
+    <xacro:create_zone parent="wall4_link" offset_x="12" offset_y="0" parent_two="wall4_link"/>
+    <xacro:create_zone parent="wall5_link" offset_x="16" offset_y="0" parent_two="wall5_link"/>
+    <xacro:create_zone parent="wall6_link" offset_x="20" offset_y="0" parent_two="wall6_link"/>
+    <xacro:create_zone parent="wall7_link" offset_x="24" offset_y="0" parent_two="wall7_link"/>
+    <xacro:create_zone parent="wall8_link" offset_x="0" offset_y="-4" parent_two="wall8_link"/>
+    <xacro:create_zone parent="wall9_link" offset_x="4" offset_y="-4" parent_two="wall9_link"/>
+    <xacro:create_zone parent="wall10_link" offset_x="8" offset_y="-4" parent_two="wall10_link"/>
+    <xacro:create_zone parent="wall11_link" offset_x="12" offset_y="-4" parent_two="wall11_link"/>
+    <xacro:create_zone parent="wall12_link" offset_x="16" offset_y="-4" parent_two="wall12_link"/>
+    <xacro:create_zone parent="wall13_link" offset_x="20" offset_y="-4" parent_two="wall13_link"/>
+    <xacro:create_zone parent="wall14_link" offset_x="24" offset_y="-4" parent_two="wall14_link"/>
+    <xacro:create_zone parent="wall15_link" offset_x="0" offset_y="-8" parent_two="wall15_link"/>
+    <xacro:create_zone parent="wall16_link" offset_x="4" offset_y="-8" parent_two="wall16_link"/>
+    <xacro:create_zone parent="wall17_link" offset_x="8" offset_y="-8" parent_two="wall17_link"/>
+    <xacro:create_zone parent="wall18_link" offset_x="12" offset_y="-8" parent_two="wall18_link"/>
+    <xacro:create_zone parent="wall19_link" offset_x="16" offset_y="-8" parent_two="wall19_link"/>
+    <xacro:create_zone parent="wall20_link" offset_x="20" offset_y="-8" parent_two="wall20_link"/>
+    <xacro:create_zone parent="wall21_link" offset_x="24" offset_y="-8" parent_two="wall21_link"/>
+    <xacro:create_zone parent="wall22_link" offset_x="0" offset_y="-12" parent_two="wall22_link"/>
+    <xacro:create_zone parent="wall23_link" offset_x="4" offset_y="-12" parent_two="wall23_link"/>
+    <xacro:create_zone parent="wall24_link" offset_x="8" offset_y="-12" parent_two="wall24_link"/>
+    <xacro:create_zone parent="wall25_link" offset_x="12" offset_y="-12" parent_two="wall25_link"/> -->
 </robot>

File: esp32_receiver/description/robot_core.xacro (robot description, xacro)
@@ -67,58 +67,110 @@
         <material>Gazebo/Orange</material>
     </gazebo>
-    <!-- ======= Left Wheel ======= -->
-    <joint name="left_wheel_joint" type="continuous">
-        <parent link="base_link"/>
-        <child link="left_wheel"/>
+    <!-- ======= front_Left Wheel ======= -->
+    <joint name="front_left_wheel_joint" type="continuous">
+        <parent link="base_link"/>
+        <child link="front_left_wheel"/>
         <origin xyz="0.05 0.06 0" rpy="-${pi/2} 0 0"/>
         <axis xyz="0 0 1"/>
     </joint>
-    <link name="left_wheel">
-        <visual>
-            <geometry>
-                <cylinder radius="0.03" length="0.02"/>
-            </geometry>
-            <material name="blue"/>
-        </visual>
-        <collision>
-            <geometry>
-                <sphere radius="0.03"/>
-            </geometry>
-        </collision>
-        <xacro:inertial_cylinder mass="0.05" length="0.02" radius="0.03">
-            <origin xyz="0 0 0" rpy="0 0 0"/>
-        </xacro:inertial_cylinder>
-    </link>
-    <gazebo reference="left_wheel">
-        <material>Gazebo/Blue</material>
-    </gazebo>
-    <!-- ======= Right Wheel ======= -->
-    <joint name="right_wheel_joint" type="continuous">
-        <parent link="base_link"/>
-        <child link="right_wheel"/>
+    <link name="front_left_wheel">
+        <visual>
+            <geometry>
+                <cylinder radius="0.03" length="0.02"/>
+            </geometry>
+            <material name="blue"/>
+        </visual>
+        <collision>
+            <geometry>
+                <sphere radius="0.03"/>
+            </geometry>
+        </collision>
+        <xacro:inertial_cylinder mass="0.05" length="0.02" radius="0.03">
+            <origin xyz="0 0 0" rpy="0 0 0"/>
+        </xacro:inertial_cylinder>
+    </link>
+    <gazebo reference="front_left_wheel">
+        <material>Gazebo/Blue</material>
+    </gazebo>
+    <!-- ======= front_Right Wheel ======= -->
+    <joint name="front_right_wheel_joint" type="continuous">
+        <parent link="base_link"/>
+        <child link="front_right_wheel"/>
         <origin xyz="0.05 -0.06 0" rpy="${pi/2} 0 0"/>
         <axis xyz="0 0 -1"/>
     </joint>
-    <link name="right_wheel">
-        <visual>
-            <geometry>
-                <cylinder radius="0.03" length="0.02"/>
-            </geometry>
-            <material name="blue"/>
-        </visual>
-        <collision>
-            <geometry>
-                <sphere radius="0.03"/>
-            </geometry>
-        </collision>
-        <xacro:inertial_cylinder mass="0.05" length="0.02" radius="0.03">
-            <origin xyz="0 0 0" rpy="0 0 0"/>
-        </xacro:inertial_cylinder>
-    </link>
-    <gazebo reference="right_wheel">
+    <link name="front_right_wheel">
+        <visual>
+            <geometry>
+                <cylinder radius="0.03" length="0.02"/>
+            </geometry>
+            <material name="blue"/>
+        </visual>
+        <collision>
+            <geometry>
+                <sphere radius="0.03"/>
+            </geometry>
+        </collision>
+        <xacro:inertial_cylinder mass="0.05" length="0.02" radius="0.03">
+            <origin xyz="0 0 0" rpy="0 0 0"/>
+        </xacro:inertial_cylinder>
+    </link>
+    <gazebo reference="front_right_wheel">
+        <material>Gazebo/Blue</material>
+    </gazebo>
+    <!-- ======= back_Right Wheel ======= -->
+    <joint name="back_right_wheel_joint" type="continuous">
+        <parent link="base_link"/>
+        <child link="back_right_wheel"/>
+        <origin xyz="-0.05 -0.06 0" rpy="${pi/2} 0 0"/>
+        <axis xyz="0 0 -1"/>
+    </joint>
+    <link name="back_right_wheel">
+        <visual>
+            <geometry>
+                <cylinder radius="0.03" length="0.02"/>
+            </geometry>
+            <material name="blue"/>
+        </visual>
+        <collision>
+            <geometry>
+                <sphere radius="0.03"/>
+            </geometry>
+        </collision>
+        <xacro:inertial_cylinder mass="0.05" length="0.02" radius="0.03">
+            <origin xyz="0 0 0" rpy="0 0 0"/>
+        </xacro:inertial_cylinder>
+    </link>
+    <gazebo reference="back_right_wheel">
+        <material>Gazebo/Blue</material>
+    </gazebo>
+    <!-- ======= back_Left Wheel ======= -->
+    <joint name="back_left_wheel_joint" type="continuous">
+        <parent link="base_link"/>
+        <child link="back_left_wheel"/>
+        <origin xyz="-0.05 0.06 0" rpy="-${pi/2} 0 0"/>
+        <axis xyz="0 0 1"/>
+    </joint>
+    <link name="back_left_wheel">
+        <visual>
+            <geometry>
+                <cylinder radius="0.03" length="0.02"/>
+            </geometry>
+            <material name="blue"/>
+        </visual>
+        <collision>
+            <geometry>
+                <sphere radius="0.03"/>
+            </geometry>
+        </collision>
+        <xacro:inertial_cylinder mass="0.05" length="0.02" radius="0.03">
+            <origin xyz="0 0 0" rpy="0 0 0"/>
+        </xacro:inertial_cylinder>
+    </link>
+    <gazebo reference="back_left_wheel">
         <material>Gazebo/Blue</material>
     </gazebo>
     <!-- ======= Caster Wheel ======= -->
-    <joint name="caster_wheel_joint" type="fixed">
+    <!-- <joint name="caster_wheel_joint" type="fixed">
         <parent link="chassis"/>
         <child link="caster_wheel"/>
@@ -145,4 +197,4 @@
         <mu1 value="0.001"/>
         <mu2 value="0.001"/>
-    </gazebo>
+    </gazebo> -->
 </robot>
