Commit message: 多機測試成功

File: esp32_receiver/urdf_data/robot.urdf (robot description, URDF)
Before this commit: robot try_gazebo, 5 links, 4 joints
Links:
- link part_1: geometry collision mesh filename=/home/u/ros2_ws/src/ros2_end/esp32_receiver/urdf_data/asset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; collision mesh filename=/home/u/ros2_ws/src/ros2_end/esp32_receiver/urdf_data/asset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
- link part_1_2: geometry collision mesh filename=/home/u/ros2_ws/src/ros2_end/esp32_receiver/urdf_data/asset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; visual mesh filename=/home/u/ros2_ws/src/ros2_end/esp32_receiver/urdf_data/asset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
- link part_1_3: geometry collision mesh filename=/home/u/ros2_ws/src/ros2_end/esp32_receiver/urdf_data/asset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; visual mesh filename=/home/u/ros2_ws/src/ros2_end/esp32_receiver/urdf_data/asset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
- link part_1_4: geometry collision mesh filename=/home/u/ros2_ws/src/ros2_end/esp32_receiver/urdf_data/asset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; visual mesh filename=/home/u/ros2_ws/src/ros2_end/esp32_receiver/urdf_data/asset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
- link part_1_5: geometry collision mesh filename=/home/u/ros2_ws/src/ros2_end/esp32_receiver/urdf_data/asset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; visual mesh filename=/home/u/ros2_ws/src/ros2_end/esp32_receiver/urdf_data/asset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
